Commit message: 更新：添加软块接触检测和力传感器数据记录功能，修改圆形运动控制器

File: franka_ros/franka_description/robots/common/franka_probe.xacro (robot description, xacro)
@@ -1,20 +1,43 @@
 <?xml version="1.0" encoding="utf-8"?>
+<!--
+  FR3机器人独立力探头定义文件
+  作者: AIRJASON50
+  日期: 2024-04-14
+  此文件定义了FR3机器人使用的力探头末端执行器。探头连接到机器人末端，
+  用于感知接触力并与环境进行交互。本文件包含探头的视觉外观、物理特性
+  和仿真参数。
+  主要修改:
+  1. 降低探头质量从1.96kg到0.5kg，使控制器能更好地控制末端姿态
+  2. 调整惯性参数与质量匹配
+  3. 添加详细的接触属性，提高力反馈准确性
+  4. 将prismatic关节改为fixed关节，使探头固定连接到机器人末端
+-->
 <robot xmlns:xacro="http://www.ros.org/wiki/xacro" name="probe">
-  <!-- 探头模型定义 -->
+  <!--
+    探头模型定义
+    参数说明:
+    - connected_to: 连接到的父链接名称
+    - arm_id: 机器人ID，用于命名链接和关节
+    - rpy: 探头相对于父链接的旋转角度(roll-pitch-yaw)
+    - xyz: 探头相对于父链接的位置偏移
+    - tcp_xyz: 工具中心点(TCP)相对于探头的位置偏移
+    - tcp_rpy: 工具中心点相对于探头的旋转角度
+    - safety_distance: 安全距离，用于碰撞检测
+    - gazebo: 是否在Gazebo中仿真
+    - description_pkg: 模型文件所在包的名称
+  -->
   <xacro:macro name="franka_probe" params="connected_to:='' arm_id:='panda' rpy:='0 0 0' xyz:='0 0 0' tcp_xyz:='0 0 0.05' tcp_rpy:='0 0 0' safety_distance:=0 gazebo:=false description_pkg:=franka_description">
     <xacro:unless value="${connected_to == ''}">
-      <!-- 使用与finger_joint类似的名称和类型 -->
-      <joint name="${arm_id}_probe_finger_joint" type="prismatic">
+      <!-- 定义探头关节 - 使用fixed类型，确保探头固定连接到机器人末端 -->
+      <joint name="${arm_id}_probe_joint" type="fixed">
         <parent link="${connected_to}" />
         <child link="${arm_id}_probe" />
         <!-- 所有情况下使用给定的位置和方向 -->
         <origin xyz="${xyz}" rpy="${rpy}" />
-        <!-- 设置为固定的prismatic关节，移动范围为0 -->
-        <axis xyz="0 0 1" />
-        <limit effort="100" lower="0.0" upper="0.0" velocity="0.2" />
-        <dynamics damping="0.3" />
       </joint>
     </xacro:unless>
+    <!-- 探头链接定义 -->
     <link name="${arm_id}_probe">
+      <!-- 视觉外观 -->
       <visual>
         <geometry>
@@ -29,4 +52,5 @@
         <origin xyz="-0.043 -0.051 -0.0" rpy="0 0 0" />
       </visual>
+      <!-- 碰撞检测几何体 -->
       <collision>
         <geometry>
@@ -52,14 +76,15 @@
         </surface>
       </collision>
+      <!-- 物理特性: 质量和惯性 -->
       <inertial>
         <!-- 原始质量：钢的密度约为7850 kg/m³，假设探头体积约为0.05×0.05×0.1=0.00025 m³ -->
-        <!-- 降低重量以减轻对控制器的负担 -->
+        <!-- 降低重量以减轻对控制器的负担，原始为1.96kg，现调整为0.5kg -->
         <mass value="0.5" />
-        <!-- 降低相应的惯性矩阵值 -->
+        <!-- 降低相应的惯性矩阵值，与质量匹配 -->
         <inertia ixx="0.0002" ixy="0" ixz="0" iyy="0.0002" iyz="0" izz="0.0001" />
         <origin xyz="-0.043 -0.051 -0.0" rpy="0 0 0" />
       </inertial>
     </link>
-    <!-- 定义探头TCP点，与末端执行器坐标系对齐 -->
+    <!-- 定义探头TCP点，与末端执行器坐标系对齐，用于力反馈和接触检测 -->
     <link name="${arm_id}_probe_tcp" />
     <joint name="${arm_id}_probe_tcp_joint" type="fixed">
@@ -68,5 +93,5 @@
       <child link="${arm_id}_probe_tcp" />
     </joint>
-    <!-- Gazebo特定标签 -->
+    <!-- Gazebo仿真特定参数 -->
     <xacro:if value="${gazebo}">
       <gazebo reference="${arm_id}_probe">
@@ -84,11 +109,11 @@
         <maxContacts>20</maxContacts>
       </gazebo>
-      <!-- 使用与finger_joint类似的名称 -->
-      <transmission name="${arm_id}_probe_finger_joint_transmission">
+      <!-- 传动系统定义 - 使用与finger_joint类似的名称 -->
+      <transmission name="${arm_id}_probe_joint_transmission">
         <type>transmission_interface/SimpleTransmission</type>
-        <joint name="${arm_id}_probe_finger_joint">
+        <joint name="${arm_id}_probe_joint">
           <hardwareInterface>hardware_interface/EffortJointInterface</hardwareInterface>
         </joint>
-        <actuator name="${arm_id}_probe_finger_joint_motor">
+        <actuator name="${arm_id}_probe_joint_motor">
           <hardwareInterface>hardware_interface/EffortJointInterface</hardwareInterface>
         </actuator>

Commit message: 更新项目进度文档和将探头颜色修改为白色

File: franka_ros/franka_description/robots/common/franka_probe.xacro (robot description, xacro)
@@ -44,6 +44,6 @@
           <mesh filename="package://${description_pkg}/meshes/probe/probe.stl" scale="0.001 0.001 0.001"/>
         </geometry>
-        <material name="red">
-          <color rgba="1 0 0 1" />
+        <material name="white">
+          <color rgba="1 1 1 1" />
         </material>
         <!-- 调整视觉模型的位置，使Z轴上表面与关节表面对齐 -->
@@ -96,5 +96,5 @@
     <xacro:if value="${gazebo}">
       <gazebo reference="${arm_id}_probe">
-        <material>Gazebo/SteelBrushed</material>
+        <material>Gazebo/White</material>
         <!-- 光滑钢材料的摩擦系数较低 -->
         <mu1>0.2</mu1>

Commit message: feat: 更新力传感器数据处理和可视化功能

File: franka_ros/franka_description/robots/common/franka_probe.xacro (robot description, xacro)
@@ -1,15 +1,16 @@
 <?xml version="1.0" encoding="utf-8"?>
 <!--
-  FR3机器人独立力探头定义文件
+  FR3机器人独立锥形力探头定义文件
   作者: AIRJASON50
-  日期: 2024-04-14
-  此文件定义了FR3机器人使用的力探头末端执行器。探头连接到机器人末端，
+  日期: 2024-05-22
+  此文件定义了FR3机器人使用的锥形力探头末端执行器。探头连接到机器人末端，
   用于感知接触力并与环境进行交互。本文件包含探头的视觉外观、物理特性
   和仿真参数。
   主要修改:
-  1. 降低探头质量从1.96kg到0.5kg，使控制器能更好地控制末端姿态
-  2. 调整惯性参数与质量匹配
-  3. 添加详细的接触属性，提高力反馈准确性
-  4. 将prismatic关节改为fixed关节，使探头固定连接到机器人末端
+  1. 视觉外观使用probe_model的STL网格模型，提供真实外观
+  2. 碰撞模型使用简化的圆柱体+球体组合，确保高效的物理仿真
+  3. 球形探针仅用于精确的接触检测，无视觉外观
+  4. STL模型坐标系调整，使探头上端（底部基座）与机器人法兰重合
+  5. 保持固定连接到机器人末端法兰
 -->
 <robot xmlns:xacro="http://www.ros.org/wiki/xacro" name="probe">
@@ -27,5 +28,5 @@
     - description_pkg: 模型文件所在包的名称
   -->
-  <xacro:macro name="franka_probe" params="connected_to:='' arm_id:='panda' rpy:='0 0 0' xyz:='0 0 0' tcp_xyz:='0 0 0.05' tcp_rpy:='0 0 0' safety_distance:=0 gazebo:=false description_pkg:=franka_description">
+  <xacro:macro name="franka_probe" params="connected_to:='' arm_id:='panda' rpy:='0 0 0' xyz:='0 0 0' tcp_xyz:='0 0 0.109' tcp_rpy:='0 0 0' safety_distance:=0 gazebo:=false description_pkg:=franka_description">
     <xacro:unless value="${connected_to == ''}">
       <!-- 定义探头关节 - 使用fixed类型，确保探头固定连接到机器人末端 -->
@@ -37,32 +38,64 @@
       </joint>
     </xacro:unless>
-    <!-- 探头链接定义 -->
+    <!-- 探头底座链接定义 - 使用STL模型外观，保持圆柱体碰撞模型 -->
     <link name="${arm_id}_probe">
-      <!-- 视觉外观 -->
+      <!-- 视觉外观 - 使用probe_model的STL网格模型 -->
       <visual>
         <geometry>
-          <mesh filename="package://${description_pkg}/meshes/probe/probe.stl" scale="0.001 0.001 0.001"/>
+          <mesh filename="package://franka_gazebo/models/probe_model/meshes/probe.stl" scale="0.001 0.001 0.001"/>
         </geometry>
-        <material name="white">
-          <color rgba="1 1 1 1" />
+        <material name="blue">
+          <color rgba="0 0 1 1" />
         </material>
-        <!-- 调整视觉模型的位置，使Z轴上表面与关节表面对齐 -->
-        <!-- STL模型的X范围：0.37-85.87，Y范围：0.64-102.12，Z范围：0-114 -->
-        <!-- 中心点约为X=43，Y=51，Z=57，但我们需要Z轴上表面对齐 -->
-        <origin xyz="-0.043 -0.051 -0.0" rpy="0 0 0" />
+        <!-- 调整STL模型位置，使模型上端（底部基座）与法兰重合，xy中心对齐 -->
+        <!-- 让探头底部与法兰对齐，Z=0位置对应法兰位置 -->
+        <origin xyz="-0.043 -0.051 0" rpy="0 0 0" />
       </visual>
-      <!-- 碰撞检测几何体 -->
+      <!-- 碰撞检测几何体 - 保持原有圆柱体模型 -->
       <collision>
         <geometry>
-          <mesh filename="package://${description_pkg}/meshes/probe/probe.stl" scale="0.001 0.001 0.001"/>
+          <cylinder radius="0.03" length="0.109"/>
         </geometry>
-        <origin xyz="-0.043 -0.051 -0.0" rpy="0 0 0" />
+        <origin xyz="0 0 0.0545" rpy="0 0 0" />
         <!-- 添加碰撞属性，提高接触精度 -->
         <surface>
           <contact>
             <ode>
-              <kp>5000000.0</kp>
-              <kd>500.0</kd>
-              <max_vel>0.1</max_vel>
+              <kp>100000.0</kp>
+              <kd>10.0</kd>
+              <max_vel>0.01</max_vel>
+              <min_depth>0.001</min_depth>
+            </ode>
+          </contact>
+          <friction>
+            <ode>
+              <mu>0.5</mu>
+              <mu2>0.5</mu2>
+            </ode>
+          </friction>
+        </surface>
+      </collision>
+      <!-- 物理特性: 质量和惯性 - 保持不变 -->
+      <inertial>
+        <mass value="0.2" />
+        <inertia ixx="0.001" ixy="0" ixz="0" iyy="0.001" iyz="0" izz="0.001" />
+        <origin xyz="0 0 0.0545" rpy="0 0 0" />
+      </inertial>
+    </link>
+    <!-- 球形探针链接定义 - 仅用于碰撞检测，无视觉外观 -->
+    <link name="${arm_id}_probe_tip">
+      <!-- 无视觉外观 - STL模型已包含完整探头形状 -->
+      <!-- 碰撞检测几何体 - 保持球形模型用于精确接触检测 -->
+      <collision>
+        <geometry>
+          <sphere radius="0.005"/>
+        </geometry>
+        <!-- 添加碰撞属性，提高接触精度 -->
+        <surface>
+          <contact>
+            <ode>
+              <kp>100000.0</kp>
+              <kd>10.0</kd>
+              <max_vel>0.01</max_vel>
               <min_depth>0.0001</min_depth>
             </ode>
@@ -70,25 +103,27 @@
           <friction>
             <ode>
-              <mu>0.2</mu>
-              <mu2>0.2</mu2>
+              <mu>0.5</mu>
+              <mu2>0.5</mu2>
             </ode>
           </friction>
         </surface>
       </collision>
-      <!-- 物理特性: 质量和惯性 -->
+      <!-- 物理特性: 质量和惯性 - 保持不变 -->
       <inertial>
-        <!-- 原始质量：钢的密度约为7850 kg/m³，假设探头体积约为0.05×0.05×0.1=0.00025 m³ -->
-        <!-- 降低重量以减轻对控制器的负担，原始为1.96kg，现调整为0.5kg -->
-        <mass value="0.5" />
-        <!-- 降低相应的惯性矩阵值，与质量匹配 -->
-        <inertia ixx="0.0002" ixy="0" ixz="0" iyy="0.0002" iyz="0" izz="0.0001" />
-        <origin xyz="-0.043 -0.051 -0.0" rpy="0 0 0" />
+        <mass value="0.01" />
+        <inertia ixx="0.0001" ixy="0" ixz="0" iyy="0.0001" iyz="0" izz="0.0001" />
       </inertial>
     </link>
-    <!-- 定义探头TCP点，与末端执行器坐标系对齐，用于力反馈和接触检测 -->
+    <!-- 固定连接圆柱体和球体 -->
+    <joint name="${arm_id}_probe_to_tip" type="fixed">
+      <parent link="${arm_id}_probe" />
+      <child link="${arm_id}_probe_tip" />
+      <origin xyz="0 0 0.109" rpy="0 0 0" />
+    </joint>
+    <!-- 定义探头TCP点，与球体探针坐标系重合，用于力反馈和接触检测 -->
     <link name="${arm_id}_probe_tcp" />
     <joint name="${arm_id}_probe_tcp_joint" type="fixed">
-      <origin xyz="${tcp_xyz}" rpy="${tcp_rpy}" />
-      <parent link="${arm_id}_probe" />
+      <origin xyz="0 0 0" rpy="${tcp_rpy}" />
+      <parent link="${arm_id}_probe_tip" />
       <child link="${arm_id}_probe_tcp" />
     </joint>
@@ -96,18 +131,28 @@
     <xacro:if value="${gazebo}">
       <gazebo reference="${arm_id}_probe">
-        <material>Gazebo/White</material>
-        <!-- 光滑钢材料的摩擦系数较低 -->
-        <mu1>0.2</mu1>
-        <mu2>0.2</mu2>
+        <material>Gazebo/Blue</material>
+        <!-- 钢材料的摩擦系数 -->
+        <mu1>0.5</mu1>
+        <mu2>0.5</mu2>
         <!-- 增加刚度和阻尼，模拟硬质钢材料 -->
-        <kp>5000000.0</kp>
-        <kd>500.0</kd>
-        <!-- 设置为物理独立，使其在Gazebo中显示为单独模型 -->
+        <kp>100000.0</kp>
+        <kd>10.0</kd>
         <selfCollide>true</selfCollide>
         <provideFeedback>true</provideFeedback>
-        <!-- 设置金属表面特性 -->
         <maxContacts>20</maxContacts>
       </gazebo>
-      <!-- 传动系统定义 - 使用与finger_joint类似的名称 -->
+      <gazebo reference="${arm_id}_probe_tip">
+        <!-- 球形探针无视觉外观，仅用于碰撞检测 -->
+        <!-- 球形探针的摩擦系数 -->
+        <mu1>0.5</mu1>
+        <mu2>0.5</mu2>
+        <!-- 增加刚度和阻尼，模拟硬质钢材料 -->
+        <kp>100000.0</kp>
+        <kd>10.0</kd>
+        <selfCollide>true</selfCollide>
+        <provideFeedback>true</provideFeedback>
+        <maxContacts>20</maxContacts>
+      </gazebo>
+      <!-- 传动系统定义 -->
       <transmission name="${arm_id}_probe_joint_transmission">
         <type>transmission_interface/SimpleTransmission</type>
